File: RemoteBoard.sch (EAGLE design)
At the start: 37 parts, among them J1 SOCKETS9111_SLOT, J2 SOCKETS9111_SLOT, J3 SOCKETS9111_SLOT, J4 CONN_42.54_SCREW, Q3 DMG3404, U1 SPG30, U2 TXS0102DCU, U3 MIC53651.8SC70, U4 BME280, U5 LTC2054, U6 MCP3221, U7 TPS7A0533DBV, U8 TCS3400

Commit message: Minor updates, part vals
Changed 1x7 connector on Primary board to 1x4 and 1x3 because 1x7 0.1" screw terminals are made of Corinthian Leather apparently, also updated part values and BoM vals
Parts:
- C1, C2, C7: device bschulz:C-EUC0805 -> bschulz_passives:C-EU1UFC0805
- C10, C11, C12: device bschulz_passives:C-EUC0805 -> bschulz_passives:C-EU1UFC0805
- C3, C4, C5: value (none) -> 0.1uF; device bschulz:C-EUC0805 -> bschulz_passives:C-EU0.1UFC0805
- C6, C8: device bschulz:C-EUC0805 -> bschulz_passives:C-EU0.1UFC0805
- C9: device bschulz_passives:C-EUC0805 -> bschulz_passives:C-EU0.1UFC0805
- R1: device bschulz_passives:R-EU_R0805 -> bschulz_passives:R-EU_100R0805
- R2: device bschulz_passives:R-EU_R0805 -> bschulz_passives:R-EU_1KR0805
- R3: device bschulz_passives:R-EU_R0805 -> bschulz_passives:R-EU_78.7KR0805
- R4: device bschulz_passives:R-EU_R0805 -> bschulz_passives:R-EU_86.6KR0805
